Commit message: controller enabled

File: dyros_canary_description/robots/dyros_canary.urdf (robot description, URDF)
Before this commit: robot dyros_canary, 31 links, 30 joints
Links:
- added link panda_left_hand; collision mesh filename=package://franka_description/meshes/collision/hand.stl; visual mesh filename=package://franka_description/meshes/visual/hand.dae
- added link panda_left_leftfinger; collision mesh filename=package://franka_description/meshes/collision/finger.stl; visual mesh filename=package://franka_description/meshes/visual/finger.dae
- added link panda_left_rightfinger; collision mesh filename=package://franka_description/meshes/collision/finger.stl; visual mesh filename=package://franka_description/meshes/visual/finger.dae
- added link panda_right_hand; collision mesh filename=package://franka_description/meshes/collision/hand.stl; visual mesh filename=package://franka_description/meshes/visual/hand.dae
- added link panda_right_leftfinger; collision mesh filename=package://franka_description/meshes/collision/finger.stl; visual mesh filename=package://franka_description/meshes/visual/finger.dae
- added link panda_right_rightfinger; collision mesh filename=package://franka_description/meshes/collision/finger.stl; visual mesh filename=package://franka_description/meshes/visual/finger.dae
Joints:
- added joint panda_left_finger_joint1: type prismatic, parent panda_left_hand, child panda_left_leftfinger, origin xyz=0 0 0.0584 rpy=0 0 0, axis 0 1 0, limit lower=-0.001 upper=0.04 effort=20 velocity=0.3
- added joint panda_left_finger_joint2: type prismatic, parent panda_left_hand, child panda_left_rightfinger, origin xyz=0 0 0.0584 rpy=0 0 0, axis 0 -1 0, limit lower=-0.001 upper=0.04 effort=20 velocity=0.3
- added joint panda_left_hand_joint: type fixed, parent panda_left_link8, child panda_left_hand, origin xyz=0 0 0 rpy=0 0 -0.7853981625
- added joint panda_right_finger_joint1: type prismatic, parent panda_right_hand, child panda_right_leftfinger, origin xyz=0 0 0.0584 rpy=0 0 0, axis 0 1 0, limit lower=-0.001 upper=0.04 effort=20 velocity=0.3
- added joint panda_right_finger_joint2: type prismatic, parent panda_right_hand, child panda_right_rightfinger, origin xyz=0 0 0.0584 rpy=0 0 0, axis 0 -1 0, limit lower=-0.001 upper=0.04 effort=20 velocity=0.3
- added joint panda_right_hand_joint: type fixed, parent panda_right_link8, child panda_right_hand, origin xyz=0 0 0 rpy=0 0 -0.7853981625
- joint panda_left_joint_top_plate_link: origin xyz=0.3058 -0.15 0.0065 rpy=0.0 0.0 -1.570796325 -> xyz=0.0289 0.1913 0.2119 rpy=-0.7853981625 0.0 0
- joint panda_right_joint_top_plate_link: origin xyz=0.3058 0.15 0.0065 rpy=0.0 0.0 1.570796325 -> xyz=0.0289 -0.1913 0.2119 rpy=0.7853981625 0.0 0

File: dyros_canary_description/robots/dyros_canary.xacro (robot description, xacro)
@@ -7,6 +7,6 @@
   <xacro:include filename="$(find franka_description)/robots/hand.xacro"/>
   <xacro:husky_robot/>
-  <xacro:panda_arm arm_id='panda_left' connected_to="top_plate_link" xyz="0.25 -0.20 0.0065" rpy="0.0 0.0 ${-pi/2}"/>
-  <xacro:panda_arm arm_id='panda_right' connected_to="top_plate_link" xyz="0.25 0.20 0.0065" rpy="0.0 0.0 ${+pi/2}"/>
+  <xacro:panda_arm arm_id='panda_left' connected_to="top_plate_link" xyz="0.0289 0.1913 0.2119" rpy="${-pi/4} 0.0 0"/>
+  <xacro:panda_arm arm_id='panda_right' connected_to="top_plate_link" xyz="0.0289 -0.1913 0.2119" rpy="${+pi/4} 0.0 0"/>
   <xacro:hand ns="panda_left" rpy="0 0 ${-pi/4}" connected_to="panda_left_link8"/>
   <xacro:hand ns="panda_right" rpy="0 0 ${-pi/4}" connected_to="panda_right_link8"/>
